File: _saved_voctoknopf1.sch (KiCad schematic (older format))
At the start: 10 parts

Commit message: case 3d file, more pcb work
Parts:
- added ARDUINO?: ARDUINO_NANO, symbol ARDUINO_NANO
- added SW? (x2): MX_D, symbol MX_D
Other:
- moved on the sheet: ARDUINO?
Changed lines of the file:
@@
 LIBS:arduino
 LIBS:microchip_pic12mcu
+LIBS:cherry
+LIBS:keyboard_components
 LIBS:voctoknopf1-cache
 EELAYER 25 0
@@
 L ARDUINO_NANO ARDUINO?
 U 1 1 5A1E84AB
-P 10250 3450
-F 0 "ARDUINO?" H 10250 4300 70  0000 C CNN
-F 1 "ARDUINO_NANO" V 10250 3450 70  0000 C CNN
-F 2 "" H 10250 3450 60  0000 C CNN
-F 3 "" H 10250 3450 60  0000 C CNN
-	1    10250 3450
+P 10250 3950
+F 0 "ARDUINO?" H 10250 4800 70  0000 C CNN
+F 1 "ARDUINO_NANO" V 10250 3950 70  0000 C CNN
+F 2 "" H 10250 3950 60  0000 C CNN
+F 3 "" H 10250 3950 60  0000 C CNN
+	1    10250 3950
+	0    -1   -1   0
+$EndComp
+$Comp
+L MX_D SW?
+U 1 1 5A1E8A84
+P 5200 1800
+F 0 "SW?" H 5200 1900 60  0000 C CNN
+F 1 "MX_D" H 5200 1800 60  0000 C CNN
+F 2 "" H 5200 1800 60  0001 C CNN
+F 3 "" H 5200 1800 60  0001 C CNN
+	1    5200 1800
 	1    0    0    -1
 $EndComp
+$Comp
+L MX_D SW?
+U 1 1 5A1E8B0E
+P 4150 1850
+F 0 "SW?" H 4150 1950 60  0000 C CNN
+F 1 "MX_D" H 4150 1850 60  0000 C CNN
+F 2 "" H 4150 1850 60  0001 C CNN
+F 3 "" H 4150 1850 60  0001 C CNN
+	1    4150 1850
+	1    0    0    -1
+$EndComp
+$Comp
+L ARDUINO_NANO ARDUINO?
+U 1 1 5A1E8DE8
+P 10250 1850
+F 0 "ARDUINO?" H 10250 2700 70  0000 C CNN
+F 1 "ARDUINO_NANO" V 10250 1850 70  0000 C CNN
+F 2 "" H 10250 1850 60  0000 C CNN
+F 3 "" H 10250 1850 60  0000 C CNN
+	1    10250 1850
+	0    -1   -1   0
+$EndComp
 $EndSCHEMATC
