File: voctoknopf1.sch (KiCad schematic (older format))
At the start: 46 parts, among them SW1 MX_D, SW2 MX_D, SW3 MX_D, U2 MCP23017, U3 MCP23017

Commit message: circuit
Parts:
- gave numbers to parts that had none: 33
- renumbered U2 to U1, U3 to U2
Connections:
- no-connect marks 0 -> 54
Other:
- note added: "StreamOn"
- note added: "TAKE"
- note added: "a"
- note added: "b"
- note added: "composite_modes"
Changed lines of the file:
@@
 $EndComp
 $Comp
-L MCP23017 U2
+L MCP23017 U1
 U 1 1 5A16E83C
 P 5000 1950
-F 0 "U2" H 4900 2975 50  0000 R CNN
+F 0 "U1" H 4900 2975 50  0000 R CNN
 F 1 "MCP23017" H 4900 2900 50  0000 R CNN
 F 2 "" H 5050 1000 50  0001 L CNN
@@
 $EndComp
 $Comp
-L MCP23017 U3
+L MCP23017 U2
 U 1 1 5A16E8C4
 P 4750 5350
-F 0 "U3" H 4650 6375 50  0000 R CNN
+F 0 "U2" H 4650 6375 50  0000 R CNN
 F 1 "MCP23017" H 4650 6300 50  0000 R CNN
 F 2 "" H 4800 4400 50  0001 L CNN
@@
 $EndComp
 $Comp
-L R R?
+L R R13
 U 1 1 5A1EDF8E
 P 2250 3450
-F 0 "R?" V 2330 3450 50  0000 C CNN
+F 0 "R13" V 2330 3450 50  0000 C CNN
 F 1 "10 k" V 2250 3450 50  0000 C CNN
 F 2 "" V 2180 3450 50  0001 C CNN
@@
 $EndComp
 $Comp
-L R R?
+L R R12
 U 1 1 5A1EDF94
 P 2050 3450
-F 0 "R?" V 2130 3450 50  0000 C CNN
+F 0 "R12" V 2130 3450 50  0000 C CNN
 F 1 "220" V 2050 3450 50  0000 C CNN
 F 2 "" V 1980 3450 50  0001 C CNN
@@
 $EndComp
 $Comp
-L R R?
+L R R15
 U 1 1 5A1EDF9A
 P 2950 3450
-F 0 "R?" V 3030 3450 50  0000 C CNN
+F 0 "R15" V 3030 3450 50  0000 C CNN
 F 1 "10 k" V 2950 3450 50  0000 C CNN
 F 2 "" V 2880 3450 50  0001 C CNN
@@
 $EndComp
 $Comp
-L R R?
+L R R14
 U 1 1 5A1EDFA0
 P 2750 3450
-F 0 "R?" V 2830 3450 50  0000 C CNN
+F 0 "R14" V 2830 3450 50  0000 C CNN
 F 1 "220" V 2750 3450 50  0000 C CNN
 F 2 "" V 2680 3450 50  0001 C CNN
@@
 $EndComp
 $Comp
-L R R?
+L R R11
 U 1 1 5A1EDFA6
 P 1550 3450
-F 0 "R?" V 1630 3450 50  0000 C CNN
+F 0 "R11" V 1630 3450 50  0000 C CNN
 F 1 "10 k" V 1550 3450 50  0000 C CNN
 F 2 "" V 1480 3450 50  0001 C CNN
@@
 $EndComp
 $Comp
-L R R?
+L R R10
 U 1 1 5A1EDFAC
 P 1350 3450
-F 0 "R?" V 1430 3450 50  0000 C CNN
+F 0 "R10" V 1430 3450 50  0000 C CNN
 F 1 "220" V 1350 3450 50  0000 C CNN
 F 2 "" V 1280 3450 50  0001 C CNN
@@
 $EndComp
 $Comp
-L MX_D SW?
+L MX_D SW5
 U 1 1 5A1EDFB2
 P 1850 2750
-F 0 "SW?" H 1850 2850 60  0000 C CNN
+F 0 "SW5" H 1850 2850 60  0000 C CNN
 F 1 "MX_D" H 1850 2750 60  0000 C CNN
 F 2 "" H 1850 2750 60  0001 C CNN
@@
 $EndComp
 $Comp
-L MX_D SW?
+L MX_D SW4
 U 1 1 5A1EDFB8
 P 1150 2750
-F 0 "SW?" H 1150 2850 60  0000 C CNN
+F 0 "SW4" H 1150 2850 60  0000 C CNN
 F 1 "MX_D" H 1150 2750 60  0000 C CNN
 F 2 "" H 1150 2750 60  0001 C CNN
@@
 $EndComp
 $Comp
-L MX_D SW?
+L MX_D SW6
 U 1 1 5A1EDFBE
 P 2550 2750
-F 0 "SW?" H 2550 2850 60  0000 C CNN
+F 0 "SW6" H 2550 2850 60  0000 C CNN
 F 1 "MX_D" H 2550 2750 60  0000 C CNN
 F 2 "" H 2550 2750 60  0001 C CNN
@@
 $EndComp
 $Comp
-L R R?
+L R R17
 U 1 1 5A1EE0D4
 P 3750 3450
-F 0 "R?" V 3830 3450 50  0000 C CNN
+F 0 "R17" V 3830 3450 50  0000 C CNN
 F 1 "10 k" V 3750 3450 50  0000 C CNN
 F 2 "" V 3680 3450 50  0001 C CNN
@@
 $EndComp
 $Comp
-L R R?
+L R R16
 U 1 1 5A1EE0DA
 P 3550 3450
-F 0 "R?" V 3630 3450 50  0000 C CNN
+F 0 "R16" V 3630 3450 50  0000 C CNN
 F 1 "220" V 3550 3450 50  0000 C CNN
 F 2 "" V 3480 3450 50  0001 C CNN
@@
 $EndComp
 $Comp
-L MX_D SW?
+L MX_D SW7
 U 1 1 5A1EE0E0
 P 3350 2750
-F 0 "SW?" H 3350 2850 60  0000 C CNN
+F 0 "SW7" H 3350 2850 60  0000 C CNN
 F 1 "MX_D" H 3350 2750 60  0000 C CNN
 F 2 "" H 3350 2750 60  0001 C CNN
@@
 $EndComp
 $Comp
-L R R?
+L R R21
 U 1 1 5A1EE44E
 P 1950 5150
-F 0 "R?" V 2030 5150 50  0000 C CNN
+F 0 "R21" V 2030 5150 50  0000 C CNN
 F 1 "10 k" V 1950 5150 50  0000 C CNN
 F 2 "" V 1880 5150 50  0001 C CNN
@@
 $EndComp
 $Comp
-L R R?
+L R R20
 U 1 1 5A1EE454
 P 1700 5150
-F 0 "R?" V 1780 5150 50  0000 C CNN
+F 0 "R20" V 1780 5150 50  0000 C CNN
 F 1 "220" V 1700 5150 50  0000 C CNN
 F 2 "" V 1630 5150 50  0001 C CNN
@@
 $EndComp
 $Comp
-L R R?
+L R R23
 U 1 1 5A1EE45A
 P 2650 5150
-F 0 "R?" V 2730 5150 50  0000 C CNN
+F 0 "R23" V 2730 5150 50  0000 C CNN
 F 1 "10 k" V 2650 5150 50  0000 C CNN
 F 2 "" V 2580 5150 50  0001 C CNN
@@
 $EndComp
 $Comp
-L R R?
+L R R22
 U 1 1 5A1EE460
 P 2400 5150
-F 0 "R?" V 2480 5150 50  0000 C CNN
+F 0 "R22" V 2480 5150 50  0000 C CNN
 F 1 "220" V 2400 5150 50  0000 C CNN
 F 2 "" V 2330 5150 50  0001 C CNN
@@
 $EndComp
 $Comp
-L R R?
+L R R19
 U 1 1 5A1EE466
 P 1250 5150
-F 0 "R?" V 1330 5150 50  0000 C CNN
+F 0 "R19" V 1330 5150 50  0000 C CNN
 F 1 "10 k" V 1250 5150 50  0000 C CNN
 F 2 "" V 1180 5150 50  0001 C CNN
@@
 $EndComp
 $Comp
-L R R?
+L R R18
 U 1 1 5A1EE46C
 P 1000 5150
-F 0 "R?" V 1080 5150 50  0000 C CNN
+F 0 "R18" V 1080 5150 50  0000 C CNN
 F 1 "220" V 1000 5150 50  0000 C CNN
 F 2 "" V 930 5150 50  0001 C CNN
@@
 $EndComp
 $Comp
-L MX_D SW?
+L MX_D SW9
 U 1 1 5A1EE472
 P 1500 4550
-F 0 "SW?" H 1500 4650 60  0000 C CNN
+F 0 "SW9" H 1500 4650 60  0000 C CNN
 F 1 "MX_D" H 1500 4550 60  0000 C CNN
 F 2 "" H 1500 4550 60  0001 C CNN
@@
 $EndComp
 $Comp
-L MX_D SW?
+L MX_D SW8
 U 1 1 5A1EE478
 P 800 4550
-F 0 "SW?" H 800 4650 60  0000 C CNN
+F 0 "SW8" H 800 4650 60  0000 C CNN
 F 1 "MX_D" H 800 4550 60  0000 C CNN
 F 2 "" H 800 4550 60  0001 C CNN
@@
 $EndComp
 $Comp
-L MX_D SW?
+L MX_D SW10
 U 1 1 5A1EE47E
 P 2200 4550
-F 0 "SW?" H 2200 4650 60  0000 C CNN
+F 0 "SW10" H 2200 4650 60  0000 C CNN
 F 1 "MX_D" H 2200 4550 60  0000 C CNN
 F 2 "" H 2200 4550 60  0001 C CNN
@@
 $EndComp
 $Comp
-L R R?
+L R R25
 U 1 1 5A1EE484
 P 3400 5150
-F 0 "R?" V 3480 5150 50  0000 C CNN
+F 0 "R25" V 3480 5150 50  0000 C CNN
 F 1 "10 k" V 3400 5150 50  0000 C CNN
 F 2 "" V 3330 5150 50  0001 C CNN
@@
 $EndComp
 $Comp
-L R R?
+L R R24
 U 1 1 5A1EE48A
 P 3150 5150
-F 0 "R?" V 3230 5150 50  0000 C CNN
+F 0 "R24" V 3230 5150 50  0000 C CNN
 F 1 "220" V 3150 5150 50  0000 C CNN
 F 2 "" V 3080 5150 50  0001 C CNN
@@
 $EndComp
 $Comp
-L MX_D SW?
+L MX_D SW11
 U 1 1 5A1EE490
 P 2950 4550
-F 0 "SW?" H 2950 4650 60  0000 C CNN
+F 0 "SW11" H 2950 4650 60  0000 C CNN
 F 1 "MX_D" H 2950 4550 60  0000 C CNN
 F 2 "" H 2950 4550 60  0001 C CNN
@@
 $EndComp
 $Comp
-L R R?
+L R R26
 U 1 1 5A1EF91E
 P 3100 6000
-F 0 "R?" V 3180 6000 50  0000 C CNN
+F 0 "R26" V 3180 6000 50  0000 C CNN
 F 1 "10 k" V 3100 6000 50  0000 C CNN
 F 2 "" V 3030 6000 50  0001 C CNN
@@
 $EndComp
 $Comp
-L R R?
+L R R27
 U 1 1 5A1EF924
 P 3600 6350
-F 0 "R?" V 3680 6350 50  0000 C CNN
+F 0 "R27" V 3680 6350 50  0000 C CNN
 F 1 "220" V 3600 6350 50  0000 C CNN
 F 2 "" V 3530 6350 50  0001 C CNN
@@
 $EndComp
 $Comp
-L MX_D SW?
+L MX_D SW12
 U 1 1 5A1EF92A
 P 3050 6300
-F 0 "SW?" H 3050 6400 60  0000 C CNN
+F 0 "SW12" H 3050 6400 60  0000 C CNN
 F 1 "MX_D" H 3050 6300 60  0000 C CNN
 F 2 "" H 3050 6300 60  0001 C CNN
@@
 GND
 $Comp
-L LED D?
+L LED D2
 U 1 1 5A2062E7
 P 8850 1400
-F 0 "D?" H 8850 1500 50  0000 C CNN
+F 0 "D2" H 8850 1500 50  0000 C CNN
 F 1 "LED" H 8850 1300 50  0000 C CNN
 F 2 "" H 8850 1400 50  0001 C CNN
@@
 $EndComp
 $Comp
-L LED D?
+L LED D1
 U 1 1 5A2063A3
 P 8450 1400
-F 0 "D?" H 8450 1500 50  0000 C CNN
+F 0 "D1" H 8450 1500 50  0000 C CNN
 F 1 "LED" H 8450 1300 50  0000 C CNN
 F 2 "" H 8450 1400 50  0001 C CNN
@@
 $EndComp
 $Comp
-L R R?
+L R R9
 U 1 1 5A2069C6
 P 9200 2950
-F 0 "R?" V 9280 2950 50  0000 C CNN
+F 0 "R9" V 9280 2950 50  0000 C CNN
 F 1 "10 k" V 9200 2950 50  0000 C CNN
 F 2 "" V 9130 2950 50  0001 C CNN
@@
 $EndComp
 $Comp
-L R R?
+L R R8
 U 1 1 5A2069CC
 P 8850 1850
-F 0 "R?" V 8930 1850 50  0000 C CNN
+F 0 "R8" V 8930 1850 50  0000 C CNN
 F 1 "220" V 8850 1850 50  0000 C CNN
 F 2 "" V 8780 1850 50  0001 C CNN
@@
 $EndComp
 $Comp
-L R R?
+L R R7
 U 1 1 5A2083E1
 P 8450 1850
-F 0 "R?" V 8530 1850 50  0000 C CNN
+F 0 "R7" V 8530 1850 50  0000 C CNN
 F 1 "220" V 8450 1850 50  0000 C CNN
 F 2 "" V 8380 1850 50  0001 C CNN
@@
 $EndComp
 $Comp
-L Conn_01x02 J?
+L Conn_01x02 J1
 U 1 1 5A20964F
 P 9400 1500
-F 0 "J?" H 9400 1600 50  0000 C CNN
+F 0 "J1" H 9400 1600 50  0000 C CNN
 F 1 "Conn_01x02" H 9400 1300 50  0000 C CNN
 F 2 "" H 9400 1500 50  0001 C CNN
@@
 	5500 1150 5500 800
 Connection ~ 5500 800
-Wire Wire Line
-	5500 2250 5700 2250
 Connection ~ 6600 1100
 Wire Wire Line
@@
 Wire Wire Line
 	9200 2800 9200 1600
+NoConn ~ 7600 4550
+NoConn ~ 7500 4550
+NoConn ~ 7400 4550
+NoConn ~ 7300 4550
+NoConn ~ 7200 4550
+NoConn ~ 7100 4550
+NoConn ~ 7000 4550
+NoConn ~ 6900 4550
+NoConn ~ 6800 4550
+NoConn ~ 6700 4550
+NoConn ~ 6600 4550
+NoConn ~ 6500 4550
+NoConn ~ 4250 6150
+NoConn ~ 4250 6050
+NoConn ~ 4250 5950
+NoConn ~ 4250 5850
+NoConn ~ 4250 5750
+NoConn ~ 4250 5650
+NoConn ~ 4500 2750
+NoConn ~ 4500 2650
+NoConn ~ 7700 1250
+NoConn ~ 7600 1250
+NoConn ~ 7500 1250
+NoConn ~ 7400 1250
+NoConn ~ 7300 1250
+NoConn ~ 7000 1250
+NoConn ~ 6900 1250
+NoConn ~ 6700 1250
+NoConn ~ 6500 1250
+NoConn ~ 6500 2450
+NoConn ~ 6600 2450
+NoConn ~ 6700 2450
+NoConn ~ 6800 2450
+NoConn ~ 6900 2450
+NoConn ~ 7000 2450
+NoConn ~ 7100 2450
+NoConn ~ 7500 2450
+NoConn ~ 7600 2450
+NoConn ~ 7700 3350
+NoConn ~ 7600 3350
+NoConn ~ 7500 3350
+NoConn ~ 7400 3350
+NoConn ~ 7300 3350
+NoConn ~ 7200 3350
+NoConn ~ 7100 3350
+NoConn ~ 7000 3350
+NoConn ~ 6900 3350
+NoConn ~ 6800 3350
+NoConn ~ 6700 3350
+NoConn ~ 6500 3350
+NoConn ~ 5250 5050
+NoConn ~ 5250 4950
+NoConn ~ 5500 1650
+NoConn ~ 5500 1550
+Wire Wire Line
+	5500 2250 5700 2250
+Text Notes 9250 1900 0    60   ~ 0
+StreamOn
+Text Notes 550  1650 0    60   ~ 0
+composite_modes
+Text Notes 600  2850 0    60   ~ 0
+a
+Text Notes 650  4900 0    60   ~ 0
+b
+Text Notes 2100 6150 0    60   ~ 0
+TAKE
 $EndSCHEMATC

Commit message: netlist
Parts:
- removed J1: Conn_01x02, symbol Conn_01x02
- added U3: CPC1017N, Buttons_Switches_SMD:SW_DIP_x2_W8.61mm_Slide_LowProfile, symbol CPC1017N
- D1, D2: footprint (none) -> LEDs:LED_D5.0mm
- R1, R10, R11, R12, R13, R14, R15, R16, R17, R18, R19, R2, R20, R21, R22, R23, R24, R25, R26, R27, R3, R4, R5, R6, R7, R8, R9: footprint (none) -> Resistors_THT:R_Axial_DIN0207_L6.3mm_D2.5mm_P7.62mm_Horizontal
- SW1, SW10, SW11, SW12, SW2, SW3, SW4, SW5, SW6, SW7, SW8, SW9: footprint (none) -> cherry:SW_PCB_4PIN
- U1, U2: footprint (none) -> Housings_DIP:DIP-28_W7.62mm_LongPads
Connections:
- net 5V: now also U3.1 (ANOD), U3.2 (CATH)
- net at ARDUINO1.8 (D5), R9.2: now also U3.3 (INOUT2), U3.4 (INOUT1)
