File: voctoknopf1.sch (KiCad schematic (older format))
At the start: 46 parts, among them SW1 MX_D, SW10 MX_D, SW11 MX_D, SW12 MX_D, SW2 MX_D, SW3 MX_D, SW4 MX_D, SW5 MX_D, SW6 MX_D, SW7 MX_D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

Commit message: scematic + netlist
Parts:
- ARDUINO1, ARDUINO2: footprint (none) -> Modules:Arduino_Nano_WithMountingHoles
Changed lines of the file:
@@
 EELAYER 25 0
 EELAYER END
-$Descr User 10237 7087
+$Descr User 10434 7284
 encoding utf-8
 Sheet 1 1
@@
 F 0 "ARDUINO2" H 7250 4800 70  0000 C CNN
 F 1 "Nano Ethernet Shield" V 7250 3950 70  0000 C CNN
-F 2 "" H 7250 3950 60  0001 C CNN
+F 2 "Modules:Arduino_Nano_WithMountingHoles" H 7250 3950 60  0001 C CNN
 F 3 "" H 7250 3950 60  0000 C CNN
 	1    7250 3950
@@
 F 0 "ARDUINO1" H 7250 2700 70  0000 C CNN
 F 1 "ARDUINO_NANO" V 7250 1850 70  0000 C CNN
-F 2 "" H 7250 1850 60  0001 C CNN
+F 2 "Modules:Arduino_Nano_WithMountingHoles" H 7250 1850 60  0001 C CNN
 F 3 "" H 7250 1850 60  0000 C CNN
 	1    7250 1850
