File: _autosave-voctoknopf1.kicad_pcb (KiCad board)
At the start: 2 copper layers, 47 parts, among them SW1 MX_D, SW10 MX_D, SW11 MX_D, SW12 MX_D, SW2 MX_D, SW3 MX_D, SW4 MX_D, SW5 MX_D, SW6 MX_D, SW7 MX_D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

Commit message: pbc work
Parts:
- moved R23 20.4 mm to (72.0, 70.5)
- moved R25 19.3 mm to (92.0, 70.8)
- moved R21 17.4 mm to (43.2, 71.0)
- moved R19 17.1 mm to (28.2, 70.5)
- moved R24 16.5 mm to (110.0, 70.5), turned to 180 degrees
- moved SW11 16.5 mm to (100.5, 83.2)
- moved R3 14.8 mm to (75.8, 22.0)
- moved R4 14.4 mm to (75.2, 15.8)
- moved R15 13.7 mm to (87.5, 54.2)
- moved R22 12.7 mm to (87.5, 78.2), turned to 270 degrees
- moved SW10 11.7 mm to (75.0, 83.2)
- moved R14 11.0 mm to (71.5, 46.5)
- moved SW6 10.9 mm to (75.0, 57.2)
- moved SW2 9.95 mm to (62.0, 19.8)
- moved R13 9.72 mm to (62.0, 61.0)
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