File: voctoknopf1.kicad_pcb (KiCad board)
At the start: 2 copper layers, 161.2 x 88.5 mm, 47 parts, among them SW1 MX_D, SW10 MX_D, SW11 MX_D, SW12 MX_D, SW2 MX_D, SW3 MX_D, SW4 MX_D, SW5 MX_D, SW6 MX_D, SW7 MX_D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

Commit message: pcb
Parts:
- moved G*** 109.7 mm to (89.8, 66.8)
Routing:
- net Net-(ARDUINO1-Pad24): track 149.4 -> 148.1 mm, vias 3 -> 4
- net Net-(ARDUINO1-Pad23): track 147.4 -> 148.7 mm, vias 3 -> 6
- net Net-(R11-Pad2): track 71.5 -> 72.1 mm, vias 2 -> 3
- added copper zone on F.Cu, net Net-(ARDUINO1-Pad16)
